File: PCBs/lab_supply_v1/line_reg.kicad_sch (KiCad schematic)
At the start: 39 parts, among them T1 EL40-PC40, U1 TOP271EG, U2 LM431ACM

Commit message: Updated PCB added current sense buffer added ADC/DAC for current/voltage sensing added ACDC converter bypass made optimal supply voltage 36 V @ 5 A
Connections:
- net +32V renamed +36V
Other:
- note added: "36 V @ 5 A"
- note removed: "32 V @ 5 A"
Changed lines of the file:
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@@
 		)
 	)
-	(text "32 V @ 5 A\n"
+	(text "36 V @ 5 A"
 		(exclude_from_sim no)
 		(at 209.296 72.39 0)
@@
 		)
 	)
+	(hierarchical_label "+36V"
+		(shape output)
+		(at 229.87 80.01 0)
+		(fields_autoplaced yes)
+		(effects
+			(font
+				(size 1.27 1.27)
+			)
+			(justify left)
+		)
+	)
 	(hierarchical_label "HOT"
 		(shape input)
@@
 		)
 	)
-	(hierarchical_label "+32V"
-		(shape output)
-		(at 229.87 80.01 0)
-		(fields_autoplaced yes)
-		(effects
-			(font
-				(size 1.27 1.27)
-				(bold yes)
-			)
-			(justify left)
-		)
-	)
